Commit message: Correct the LiDAR to a YDLIDAR X3 and build the map with SLAM
The map Nav2 ships with is now produced by SLAM Toolbox driving through the
world, not derived analytically. Getting there needed three fixes, found by
logging the Gazebo ground-truth pose alongside odometry and the SLAM estimate
throughout a 90 m run.

LiDAR
- The SDF modelled a 3.5 m HLS-LFCD LDS while the README documented a 12 m
  RPLidar A1. The robot actually carries a YDLIDAR X3, so the sensor is now
  0.12-8 m, 420 samples per revolution (0.857 deg), 7 Hz, with the scan spanning
  -pi to +pi the way ydlidar_ros2_driver publishes it. Range is what dominated
  map quality: the building is 14 m across, and at 3.5 m the scan matcher
  regularly had no reference along one axis.
- AMCL laser_max_range, both costmap raytrace/obstacle ranges and SLAM's
  max_laser_range follow the sensor. The local costmap stops at 6 m because its
  rolling window is only 6 x 6 m.

Wheel friction
- The wheels had isotropic friction (mu = mu2 = 1). With four wheels that made
  the robot resist yaw so hard it turned about 65% of the commanded rate while
  the DiffDrive plugin integrated 100% of it. fdir1 now points along the wheel
  axle, which does not rotate as the wheel spins, so mu is the sideways scrub
  coefficient and mu2 the rolling one. Dropping scrub friction makes the
  skid-steer behave like a true differential drive.
- wheel_separation 0.265 -> 0.1679, recalibrated for the new friction against
  the ground-truth pose. Yaw error is now within 3% from 0.1 to 1.0 rad/s and
  straight-line odometry is exact at every speed; before, the error was -35% and
  varied with angular velocity.

Self-similar floor plan
- Four identical columns evenly spaced every 3 m, mirrored seating and two
  identically furnished offices meant different places produced nearly identical
  scans. That fed false loop closures into the pose graph and the map came out
  with duplicated walls and columns. Columns now have irregular radii and
  spacing, the reception furniture is asymmetric, and the two offices are laid
  out differently. The meeting table is 2.6 m rather than 3.0 so the aisles
  beside it are 1.2 m instead of 0.9.
- loop_match_maximum_variance_coarse 3.0 -> 0.5 and loop_search_maximum_distance
  3.0 -> 2.0. A false closure teleported the pose by exactly the search radius,
  so capping it caps the damage.

Tooling
- Add axioma_slam/scripts/score_map.py, which scores a SLAM map against the
  exact floor plan: how far each occupied cell sits from a real obstacle, and
  how many real obstacles the map actually marks.
- generate_office_world.py now writes maps/ground_truth.{pgm,yaml} instead of
  mapa.*, so regenerating the world no longer overwrites the SLAM map.
- save_map.launch.py defaulted to the install/ share directory, where the next
  colcon build would overwrite the map. It now resolves the symlink back into
  src/ when the workspace is built with --symlink-install.

Results, all measured against the Gazebo ground-truth pose:
- SLAM map score 99.4/100. 99.8% of occupied cells within 10 cm of a real
  obstacle, nothing beyond 50 cm, 99.6% of real obstacles found within 10 cm.
- SLAM pose error 0.038 m mean, 0.18 m max, while raw odometry drifts to 4.13 m.
- Navigation on that map: 5/5 goals, zero recovery behaviours, every goal within
  0.16 m, and 21-40 s per leg against 38-57 s before.

File: src/axioma_description/urdf/axioma.urdf (robot description, URDF)
Before this commit: robot axioma_v2, 7 links, 6 joints
Links:
- link base_scan: geometry collision cylinder length=0.041 radius=0.031; visual cylinder length=0.041 radius=0.031

Commit message: Add base_footprint as the URDF root and point the stack at it
robot_state_publisher warned on every single start:

  The root link base_link has an inertia specified in the URDF, but KDL does
  not support a root link with an inertia.

Fixed the way the warning itself suggests, with a massless root link, but
base_footprint is worth having for its own sake rather than just to silence a
message.

  map -> odom -> base_footprint -> base_link -> {base_scan, imu_link, wheels}

The offset between base_footprint and base_link is -2.58 mm in z, and it is not
a fudge: wheel centres sit at z = 0.04068 while the wheels have radius 0.0381,
so with the wheels on the floor base_link ends up 0.0381 - 0.04068 below it.
Gazebo reports exactly that z for the spawned model.

That also makes odometry honest. The DiffDrive plugin publishes planar odometry
at z = 0, which is the floor, so odom_to_tf now attaches it to base_footprint
instead of base_link. It has to: base_link already hangs off base_footprint
through the URDF's fixed joint, and a frame can only have one parent, so
publishing odom -> base_link would have fought robot_state_publisher for it.
A side effect is that map -> base_scan now reports 0.14742 m, the LiDAR's real
height above the floor, where before it read a flat 0.15.

Followed through everywhere the frame is named: AMCL base_frame_id,
bt_navigator, both costmaps, behavior_server and SLAM Toolbox's base_frame.

Two more things found on the way:
- axioma.urdf gave base_link 1.0 kg with a tensor that did not match the 5.0 kg
  in model.sdf. Only robot_state_publisher reads the URDF and it ignores
  inertias, so nothing was broken, but the two files disagreed. Now they match.
- slam.rviz had Fixed Frame set to base_link while showing a Map display, so
  during mapping the map slid around under the robot instead of staying put.
  It is map now. display.rviz follows base_footprint.

Verified: startup log completely clean, no warnings at all; TF resolves with one
parent per frame; navigation 5/5 with no recovery behaviours, every goal within
0.14 m of the requested pose.

File: src/axioma_description/urdf/axioma.urdf (robot description, URDF)
Before this commit: robot axioma_v2, 7 links, 6 joints
Links:
- added link base_footprint
- link base_link: mass 1.0 -> 5.0
Joints:
- added joint base_footprint_joint: type fixed, parent base_footprint, child base_link, origin xyz=0 0 -0.00258 rpy=0 0 0

Commit message: Reposition imu_link onto the chassis and document it as a design reservation
imu_link sat at (0.1, 0.1, 0.12): 4 mm past the chassis front face and 14 mm
past the left one, since the visual mesh spans x in [-0.100, 0.096] and y in
[-0.111, 0.086]. Moved it to (0, 0, 0.12), on the yaw axis directly above
base_link's origin, so a turn in place shows up as yaw rate alone rather than
centripetal acceleration a future filter would have to model.

No sensor exists in model.sdf yet, so the frame is still unused; documented
that on purpose in the URDF, control.md (with the three steps to wire it up:
an IMU sensor in the SDF, an /imu bridge, and a robot_localization EKF), and
cinematica.md's TF tree.

File: src/axioma_description/urdf/axioma.urdf (robot description, URDF)
Before this commit: robot axioma_v2, 8 links, 7 joints
Joints:
- joint imu_joint: origin xyz=0.1 0.1 0.12 rpy=0 0 0 -> xyz=0 0 0.12 rpy=0 0 0
