Commit message: Add attitude-aware localisation, a ZED 2i, and a rough-terrain world
The wheel odometry assumes the floor is flat. Drive up a ramp and it reports
z = 0 and zero pitch the whole way, so the pose diverges silently in exactly
the situation a map would need it most.

This adds the sensing and the filter that fix it, plus a world that makes the
failure visible.

- axioma_perception: a robot_localization EKF publishing odom -> base_footprint.
  ekf_sim.yaml fuses the chassis IMU for absolute roll and pitch and the wheel
  plugin for body velocity; ekf_zed.yaml is the physical-robot counterpart,
  where the ZED supplies position and yaw and the wheels are dropped entirely.
  two_d_mode stays false, since flattening z, roll and pitch would be an
  expensive way to reproduce the error the filter exists to remove. IMU yaw is
  deliberately not fused: there is no magnetometer on this robot, and the
  simulated orientation is ground truth in disguise, so fusing it would make
  the simulation look better than the hardware ever will be. Heading drift is
  SLAM Toolbox's and AMCL's problem one level up.

- axioma.urdf becomes axioma.urdf.xacro and carries a ZED 2i mounted at
  (0.098, 0, 0.10) on base_link. The camera contributes eight frames whose
  offsets follow from its geometry, and as literals they would need rederiving
  by hand every time it moves. The macro is vendored from Stereolabs and
  trimmed to the zed2i branch, with the three changes documented in its
  header. All three loaders now render it through xacro first.

- model.sdf gains a real IMU on imu_link and an RGBD camera for the ZED. Both
  worlds load gz-sim-imu-system; without it an IMU sensor publishes nothing
  and Gazebo gives no warning.

- terrain.world, emitted together with its ground-truth map from one geometry
  listing so the two cannot drift apart: an 18 x 10 m bay at z = 0 and a yard
  at z = 0.28, joined by two 8.21 deg ramps forming a closed circuit. The yard
  is split into asphalt, dirt and sand patches with genuinely different
  friction, not just different colours, which is what makes control.md's
  warning about the effective track width testable. No steps anywhere, by
  design: 3.81 cm wheels on a rigid chassis without suspension do not climb a
  riser, they hit it. _check_layout() refuses to emit the world if anything
  blocks either ramp approach or if two obstacles overlap.

- terrain_demo.launch.py brings up Gazebo, RViz and the teleop GUI together,
  with use_ekf:=false available for the contrast.

Driving straight up the north ramp onto the platform, against ground truth:
wheel odometry reports z = 0.000 m (280 mm low) and 0.00 deg of pitch, while
the EKF reports 0.286 m and -8.21 deg. On flat ground the two agree to within
3 mm over 4 m, so the filter costs nothing where it is not needed.

The EKF covariances stay at their defaults on purpose, and the YAML comments
say why: the right values depend on how much the wheels slip on each surface,
and hand-writing a 15x15 matrix before measuring that would look authoritative
without being backed by anything. The three friction patches are there to make
that measurement possible.

Also drops *.xml from .gitignore. It was meant for colcon test output, which
lands in build/ and log/ and is ignored there already, but it silently
swallowed every package manifest, axioma_perception/package.xml included,
which would have shipped the new package unbuildable.

File: src/axioma_description/urdf/axioma.urdf.xacro (robot description, xacro)
@@ -1,4 +1,18 @@
 <?xml version="1.0"?>
-<robot name="axioma_v2">
+<robot name="axioma_v2" xmlns:xacro="http://wiki.ros.org/xacro">
+  <!-- This description is xacro, not plain URDF, for exactly one reason: the
+       ZED 2i contributes eight frames whose offsets come from the camera's
+       geometry, and writing them out by hand as literal numbers would mean
+       re-deriving them by hand every time the camera moves on the chassis.
+       Everything else below is still ordinary URDF.
+       Anything that loads this file must run it through xacro first —
+       open(...).read() gets you a document full of ${...} that KDL rejects.
+       Both launch files in this repo already do (display.launch.py and
+       axioma_gazebo/launch/simulation.launch.py). -->
+  <!-- Relative, not $(find axioma_description)/urdf/..., so the file renders
+       straight out of the source tree before the package has ever been built.
+       xacro resolves a relative include against the including file, so this
+       keeps working unchanged from install/share as well. -->
+  <xacro:include filename="zed2i_macro.urdf.xacro"/>
   <!-- Base Footprint: the ground projection of base_link, and the root of the
        tree. It carries no <inertial> on purpose: KDL cannot handle an inertia
@@ -197,3 +211,26 @@
     <origin xyz="0 0 0.12" rpy="0 0 0"/>
   </joint>
+  <!-- ==================== ZED 2i ==================== -->
+  <!-- Stereo depth camera, mounted looking forward off the front face of the
+       chassis. Its job on this robot is not obstacle detection: it feeds the
+       EKF in axioma_perception with a visual-inertial pose, so that a rigid
+       4WD skid-steer with no suspension still knows where it is when the
+       wheels slip or the ground tilts. See axioma_perception/config/.
+       Mount pose. x = 0.098 puts the tripod screw at the front face of the
+       chassis (the visual mesh spans x in [-0.100, 0.096]); z = 0.10 clears
+       the deck and keeps the lenses below the LiDAR plane at z = 0.15, so the
+       camera body never shows up in the scan. rpy is zero — the 2i's base is
+       flat and the mount is not tilted, so the optical axis is horizontal.
+       The 2i is 175 mm wide on a 220 mm chassis, so it overhangs by about
+       25 mm per side. That is intentional and was checked in RViz: the stereo
+       baseline is fixed at 120 mm by the hardware, and narrowing the mount
+       would not change it.
+       Moving the camera means changing this joint and nothing else. The eight
+       frames below it, including the optical ones, follow automatically. -->
+  <xacro:zed2i_camera name="zed2i"/>
+  <joint name="zed2i_mount_joint" type="fixed">
+    <parent link="base_link"/>
+    <child link="zed2i_camera_link"/>
+    <origin xyz="0.098 0 0.10" rpy="0 0 0"/>
+  </joint>
 </robot>
